File: pcb/biosensor/biosensor.kicad_sch (KiCad schematic)
At the start: 34 parts, among them J1 Screw_Terminal_01x03, J2 Conn_01x02_Female, P1 USB_C_Plug_USB2.0, SW1 SW_DIP_x01, U1 DW01, U2 TP4056, U3 FS8205A, U4 LM2621

Commit message: pcb files
Connections:
- net Vout: now also A1.30 (VIN); no longer A1.27 (+5V)
Changed lines of the file:
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@@
   (junction (at 128.27 185.42) (diameter 0) (color 0 0 0 0)
   )
-  (junction (at 241.3 129.54) (diameter 0) (color 0 0 0 0)
-  )
   (junction (at 138.43 63.5) (diameter 0) (color 0 0 0 0)
   )
@@
   )
   (junction (at 207.01 81.28) (diameter 0) (color 0 0 0 0)
+  )
+  (junction (at 241.3 121.92) (diameter 0) (color 0 0 0 0)
   )
   (junction (at 237.49 25.4) (diameter 0) (color 0 0 0 0)
@@
     (stroke (width 0) (type default) (color 0 0 0 0))
   )
-  (wire (pts (xy 241.3 129.54) (xy 241.3 139.7))
+  (wire (pts (xy 241.3 121.92) (xy 241.3 139.7))
     (stroke (width 0) (type default) (color 0 0 0 0))
   )
@@
     (stroke (width 0) (type default) (color 0 0 0 0))
   )
+  (wire (pts (xy 241.3 121.92) (xy 245.11 121.92))
+    (stroke (width 0) (type default) (color 0 0 0 0))
+  )
   (wire (pts (xy 95.25 46.99) (xy 95.25 39.37))
     (stroke (width 0) (type default) (color 0 0 0 0))
@@
     (stroke (width 0) (type default) (color 0 0 0 0))
   )
-  (wire (pts (xy 241.3 129.54) (xy 245.11 129.54))
-    (stroke (width 0) (type default) (color 0 0 0 0))
-  )
   (wire (pts (xy 229.87 76.2) (xy 237.49 76.2))
     (stroke (width 0) (type default) (color 0 0 0 0))
@@
     (stroke (width 0) (type default) (color 0 0 0 0))
   )
-  (wire (pts (xy 231.14 129.54) (xy 241.3 129.54))
+  (wire (pts (xy 231.14 121.92) (xy 241.3 121.92))
     (stroke (width 0) (type default) (color 0 0 0 0))
   )
@@
     (effects (font (size 1.27 1.27)) (justify left bottom))
   )
-  (label "Vout" (at 245.11 129.54 0)
-    (effects (font (size 1.27 1.27)) (justify left bottom))
-  )
+  (label "Vout" (at 245.11 121.92 0)
+    (effects (font (size 1.27 1.27)) (justify left bottom))
+  )

Commit message: before esp change
Other:
- note added: "Arduino Nano BLE met sensor"
- note removed: "Arduino Nano met sensor"
Changed lines of the file:
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@@
     (effects (font (size 1.27 1.27)) (justify left bottom))
   )
-  (text "Arduino Nano met sensor" (at 152.4 104.14 0)
+  (text "Arduino Nano BLE met sensor" (at 152.4 104.14 0)
     (effects (font (size 1.27 1.27)) (justify left bottom))
   )

Commit message: massive update to pcb
Parts:
- removed A1: Arduino_Nano_v3.x, Module:Arduino_Nano, symbol MCU_Module:Arduino_Nano_v3.x
- added C10, C14: 1µF/16V(10%), symbol Device:C
- added C11, C12: 22pF/50V/(5%)(NC), symbol Device:C
- added C13: 10µF/25V/(20%), symbol Device:C
- added C15, C17, C8: 10µF/25V(20%), symbol Device:C
- added C16, C18, C9: 0.1µF/50V(10%), symbol Device:C
- added C19, C20: 0.1µF/50V(10%)(NC), symbol Device:C
- added C21: 10µF, symbol Device:C
- added D10: Opladen, symbol Device:LED
- added D11: Klaar, symbol Device:LED
- added D4: 1N5819HW-7-F, symbol Device:D
- added D5, D6, D7: LESD5D.0CT1G, Diode_SMD:D_SOD-523, symbol Diode:ESD131-B1-W0201
- added D8: SK6812MINI, LED_SMD:LED_SK6812MINI_PLCC4_3.5x3.5mm_P1.75mm, symbol LED:SK6812MINI
- added D9: 0805 RED, symbol Device:LED
- added P2: USB_C_Plug_USB2.0, Connector_USB:USB_C_Receptacle_HRO_TYPE-C-31-M-12, symbol Connector:USB_C_Plug_USB2.0
- added Q1, Q2: L8050QLT1G, symbol Simulation_SPICE:NPN
- added R11, R12, R23, R24: 10K(1%), symbol Device:R
- added R13, R16, R17, R18, R25: 0(1%), symbol Device:R
- added R14, R15: 0(1%)(NC), symbol Device:R
- added R19: 22.1K(1%), symbol Device:R
- added R20: 47.5K(1%), symbol Device:R
- added R21: 1K(1%), symbol Device:R
- added R22: 10K(1%)(NC), symbol Device:R
- added R26: 5.1K(1%), symbol Device:R
- added R27: 270K, symbol Device:R
- added R28, R30: 100K, symbol Device:R
- added R29: 1K, symbol Device:R
- added SW2, SW3: SW_Push, symbol Switch:SW_Push
- added TH1: 16K, symbol Device:Thermistor_NTC
- added U5: ESP32-C3-MINI-1, Espressif:ESP32-C3-MINI-1, symbol Espressif:ESP32-C3-MINI-1
- added U6: CP2102N-Axx-xQFN28, Package_DFN_QFN:QFN-28-1EP_5x5mm_P0.5mm_EP3.35x3.35mm, symbol Interface_USB:CP2102N-Axx-xQFN28
- added U7: SGM2212-3.3XKC3G/TR, Package_TO_SOT_SMD:SOT-223-3_TabPin2, symbol Regulator_Linear:AMS1117-3.3
- added U8: MCP73871, Package_DFN_QFN:QFN-20-1EP_4x4mm_P0.5mm_EP2.5x2.5mm, symbol Battery_Management:MCP73871
Connections:
- net BAT+: no longer J2.1 (Pin_1)
- net BAT-: no longer J2.2 (Pin_2)
- net GND: now also J2.1 (Pin_1), C10.2, C11.2, C12.2, C13.2, C14.2, C15.2, C16.2, C17.2, C18.2, C19.1, C20.1, C21.2, C8.2, C9.2, D5.1 (A1), D6.1 (A1), D7.1 (A1), D8.2 (VSS), D9.1 (K), P2.A1 (GND), P2.A12 (GND), P2.B1 (GND), P2.B12 (GND), P2.S1 (SHIELD), R20.2, R22.2, R28.2, R29.2, R30.2, SW2.2, SW3.2, TH1.1, U5.1 (GND), U5.11 (GND), U5.14 (GND), U5.2 (GND), U5.36 (GND), U5.37 (GND), U5.38 (GND), U5.39 (GND), U5.40 (GND), U5.41 (GND), U5.42 (GND), U5.43 (GND), U5.44 (GND), U5.45 (GND), U5.46 (GND), U5.47 (GND), U5.48 (GND), U5.49 (GND), U5.50 (GND), U5.51 (GND), U5.52 (GND), U5.53 (GND), U6.29 (GND), U6.3 (GND), U7.1 (GND), U8.10 (V_{SS}), U8.11 (V_{SS}), U8.21 (V_{SS})
- net OUTVCC: no longer C4.1, L1.1
- net Vout: no longer J1.1 (Pin_1)
- net GPIO4: now reaches J1.2 (Pin_2)
- net GPIO4: now also U5.18 (GPIO4/ADC1_CH4)
- new net: D6.2 (A2), P2.A7 (D-), R13.1, R14.1
- new net: C21.1, J2.2 (Pin_2), U8.14 (V_{BAT}), U8.15 (V_{BAT}), U8.16 (V_{BAT_SENSE})
- new net: R30.1, U8.12 (PROG3)
- new net: R29.1, U8.13 (PROG1)
- new net: Q2.2 (B), R24.2
- new net: D9.2 (A), R26.2
- new net: Q1.2 (B), R23.2
- new net: R21.2, U6.9 (~{RST})
- new net: R22.1, U6.11 (~{SUSPEND})
- new net: R27.2, R28.1, U8.2 (VPCC)
- new net: D7.2 (A2), P2.A6 (D+), R15.1, R16.1
- new net: C14.1, R19.2, R20.1, U6.8 (VBUS)
- new net: TH1.2, U8.5 (THERM)
- new net: R18.1, U6.25 (RXD)
- new net: R17.1, U6.26 (TXD)
- new net: D11.1 (K), U8.7 (STAT2)
- new net: D10.1 (K), U8.8 (STAT1/~{LBO})
- new net +3.3V: C8.1, C9.1, R11.2, R12.2, U5.3 (3V3)
- new net +3V3: C13.1, C17.1, C18.1, D8.4 (VDD), R21.1, U6.6 (VDD), U6.7 (VREGIN), U7.2 (VO)
- new net +5V: C15.1, C16.1, D4.1 (K), J1.1 (Pin_1), R26.1, U7.3 (VI)
- new net CHIP_PU: C10.1, C20.2, Q1.1 (C), R11.1, SW3.1, U5.8 (EN/CHIP_PU)
- new net DTR: Q2.3 (E), R23.1, U6.28 (~{DTR})
- new net GPIO0: U5.12 (GPIO0/ADC1_CH0/XTAL_32K_P)
- new net GPIO1: U5.13 (GPIO1/ADC1_CH1/XTAL_32K_N)
- new net GPIO10: U5.16 (GPIO10)
- new net GPIO18: C11.1, R14.2, U5.26 (GPIO18/USB_D-)
- new net GPIO19: C12.1, R15.2, U5.27 (GPIO19/USB_D+)
- new net GPIO5: U5.19 (GPIO5/ADC2_CH0)
- new net GPIO6: U5.20 (GPIO6)
- new net GPIO7: U5.21 (GPIO7)
- new net GPIO8: R12.1, R25.1, U5.22 (GPIO8)
- new net GPIO9: C19.2, Q2.1 (C), SW2.1, U5.23 (GPIO9)
- new net Load: C4.1, L1.1, U8.1 (OUT), U8.20 (OUT)
- new net RGB_CTRL: D8.3 (DIN), R25.2
- new net RTS: Q1.3 (E), R24.1, U6.24 (~{RTS})
- new net U0RXD: R17.2, U5.30 (GPIO20/U0RXD)
- new net U0TXD: R18.2, U5.31 (GPIO21/U0TXD)
- new net USB_DN: R13.2, U6.5 (D-)
- new net USB_DP: R16.2, U6.4 (D+)
- new net VBUS: D10.2 (A), D11.2 (A), D4.2 (A), D5.2 (A2), P2.A4 (VBUS), P2.A9 (VBUS), P2.B4 (VBUS), P2.B9 (VBUS), R19.1, R27.1, U8.17 (CE), U8.18 (IN), U8.19 (IN), U8.3 (SEL), U8.4 (PROG2), U8.9 (~{TE})
- no-connect marks 7 -> 9
Other:
- note added: "Batterijmanagement"
- note added: "ESP32"
- note added: "In schematic file van ESP staan DTR en RTS zonder invert"
- note added: "Low Dropout Regulator (LDO) en Boot- en Reset switches, status LED"
- note added: "RGB LED"
- note added: "Schroefaansluiting voor sensor"
- note added: "Serial Signal handling"
- note added: "TOODOO 5V afscheiden van VBUS, en achter Buckboost steken Vbussen naar 5V vervangen zodat het allemaal op batterij werkt"
- note added: "USB-C Ingang"
- note added: "USB-UART Bridge"
- note removed: "Arduino Nano BLE met sensor"
- moved on the sheet: C4, C5, C6, C7, D3, H1, H2, H3, H4, J1, J2, L1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

Commit message: final update?
Parts:
- removed C1, C3: 0.1uF, Capacitor_SMD:C_0805_2012Metric_Pad1.18x1.45mm_HandSolder, symbol Device:C
- removed C2: 10uF, Capacitor_SMD:C_0805_2012Metric_Pad1.18x1.45mm_HandSolder, symbol Device:C
- removed D1: RED, LED_SMD:LED_0805_2012Metric_Pad1.15x1.40mm_HandSolder, symbol Device:LED
- removed D2: GREEN, LED_SMD:LED_0805_2012Metric_Pad1.15x1.40mm_HandSolder, symbol Device:LED
- removed D4: 1N5819HW-7-F, symbol Device:D
- removed P1: USB_C_Plug_USB2.0, Connector_USB:USB_C_Receptacle_HRO_TYPE-C-31-M-12, symbol Connector:USB_C_Plug_USB2.0
- removed R1: 100, Resistor_SMD:R_0805_2012Metric_Pad1.20x1.40mm_HandSolder, symbol Device:R
- removed R2, R4, R5: 1k, Resistor_SMD:R_0603_1608Metric_Pad0.98x0.95mm_HandSolder, symbol Device:R
- removed R3: 10k, Resistor_SMD:R_0805_2012Metric_Pad1.20x1.40mm_HandSolder, symbol Device:R
- removed R6: 0R, Resistor_SMD:R_1206_3216Metric_Pad1.30x1.75mm_HandSolder, symbol Device:R
- removed U1: DW01, Package_TO_SOT_SMD:SOT-23-6_Handsoldering, symbol dw01:DW01
- removed U2: TP4056, Package_SO:SOIC-8-1EP_3.9x4.9mm_P1.27mm_EP2.29x3mm, symbol tp4056:TP4056
- removed U3: FS8205A, Package_TO_SOT_SMD:SOT-23-6_Handsoldering, symbol fs8205:FS8205A
- added D8: 1N5819HW-7-F, Diode_SMD:D_SOD-123, symbol Device:D
- C1: renamed from C4; footprint Capacitor_SMD:C_2225_5664Metric_Pad1.80x6.60mm_HandSolder -> Capacitor_SMD:C_0603_1608Metric_Pad1.08x0.95mm_HandSolder
- C10: renamed from C13; footprint (none) -> Capacitor_SMD:C_0603_1608Metric_Pad1.08x0.95mm_HandSolder
- C11: renamed from C10; footprint (none) -> Capacitor_SMD:C_0603_1608Metric_Pad1.08x0.95mm_HandSolder
- C12: renamed from C14; footprint (none) -> Capacitor_SMD:C_0603_1608Metric_Pad1.08x0.95mm_HandSolder
- C13: renamed from C15; footprint (none) -> Capacitor_SMD:C_0603_1608Metric_Pad1.08x0.95mm_HandSolder
- C14: renamed from C16; footprint (none) -> Capacitor_SMD:C_0603_1608Metric_Pad1.08x0.95mm_HandSolder
- C15: renamed from C18; footprint (none) -> Capacitor_SMD:C_0603_1608Metric_Pad1.08x0.95mm_HandSolder
- C16: renamed from C17; footprint (none) -> Capacitor_SMD:C_0603_1608Metric_Pad1.08x0.95mm_HandSolder
- C17: renamed from C19; footprint (none) -> Capacitor_SMD:C_0603_1608Metric_Pad1.08x0.95mm_HandSolder
- C18: renamed from C20; footprint (none) -> Capacitor_SMD:C_0603_1608Metric_Pad1.08x0.95mm_HandSolder
- C2: renamed from C5; footprint Capacitor_SMD:C_2225_5664Metric_Pad1.80x6.60mm_HandSolder -> Capacitor_SMD:C_0603_1608Metric_Pad1.08x0.95mm_HandSolder
- C4: renamed from C21; footprint (none) -> Capacitor_SMD:C_0603_1608Metric_Pad1.08x0.95mm_HandSolder
- C5: renamed from C7; footprint Capacitor_SMD:C_0805_2012Metric_Pad1.18x1.45mm_HandSolder -> Capacitor_SMD:C_0603_1608Metric_Pad1.08x0.95mm_HandSolder
- C6: renamed from C11; footprint (none) -> Capacitor_SMD:C_0603_1608Metric_Pad1.08x0.95mm_HandSolder
- C7: renamed from C12; footprint (none) -> Capacitor_SMD:C_0603_1608Metric_Pad1.08x0.95mm_HandSolder
- C8, C9: footprint (none) -> Capacitor_SMD:C_0603_1608Metric_Pad1.08x0.95mm_HandSolder
- D2: renamed from D10; footprint (none) -> LED_SMD:LED_0805_2012Metric_Pad1.15x1.40mm_HandSolder
- D3: renamed from D11; footprint (none) -> LED_SMD:LED_0805_2012Metric_Pad1.15x1.40mm_HandSolder
- D9: value 0805 RED -> RED; footprint (none) -> LED_SMD:LED_0805_2012Metric_Pad1.15x1.40mm_HandSolder
- Q1, Q2: footprint (none) -> Package_TO_SOT_SMD:SOT-23
- R1: renamed from R27; footprint (none) -> Resistor_SMD:R_0603_1608Metric_Pad0.98x0.95mm_HandSolder
- R10: renamed from R16; footprint (none) -> Resistor_SMD:R_0603_1608Metric_Pad0.98x0.95mm_HandSolder
- R11: renamed from R9; footprint Resistor_SMD:R_0805_2012Metric_Pad1.20x1.40mm_HandSolder -> Resistor_SMD:R_0603_1608Metric_Pad0.98x0.95mm_HandSolder
- R12: renamed from R10; footprint Resistor_SMD:R_0603_1608Metric -> Resistor_SMD:R_0603_1608Metric_Pad0.98x0.95mm_HandSolder
- R13: renamed from R11; footprint (none) -> Resistor_SMD:R_0603_1608Metric_Pad0.98x0.95mm_HandSolder
- R14: renamed from R21; footprint (none) -> Resistor_SMD:R_0603_1608Metric_Pad0.98x0.95mm_HandSolder
- R15: renamed from R17; footprint (none) -> Resistor_SMD:R_0603_1608Metric_Pad0.98x0.95mm_HandSolder
- R16: renamed from R18; footprint (none) -> Resistor_SMD:R_0603_1608Metric_Pad0.98x0.95mm_HandSolder
- R17: renamed from R23; footprint (none) -> Resistor_SMD:R_0603_1608Metric_Pad0.98x0.95mm_HandSolder
- R18: renamed from R19; footprint (none) -> Resistor_SMD:R_0603_1608Metric_Pad0.98x0.95mm_HandSolder
- R19: renamed from R22; footprint (none) -> Resistor_SMD:R_0603_1608Metric_Pad0.98x0.95mm_HandSolder
- R20, TH1: footprint (none) -> Resistor_SMD:R_0603_1608Metric_Pad0.98x0.95mm_HandSolder
- R21: renamed from R24; footprint (none) -> Resistor_SMD:R_0603_1608Metric_Pad0.98x0.95mm_HandSolder
- R22: renamed from R12; footprint (none) -> Resistor_SMD:R_0603_1608Metric_Pad0.98x0.95mm_HandSolder
- R23: renamed from R25; footprint (none) -> Resistor_SMD:R_0603_1608Metric_Pad0.98x0.95mm_HandSolder
- R24: renamed from R26; footprint (none) -> Resistor_SMD:R_0603_1608Metric_Pad0.98x0.95mm_HandSolder
- R3: renamed from R28; footprint (none) -> Resistor_SMD:R_0603_1608Metric_Pad0.98x0.95mm_HandSolder
- R5: renamed from R29; footprint (none) -> Resistor_SMD:R_0603_1608Metric_Pad0.98x0.95mm_HandSolder
- R6: renamed from R13; footprint (none) -> Resistor_SMD:R_0603_1608Metric_Pad0.98x0.95mm_HandSolder
- R7: renamed from R14; footprint (none) -> Resistor_SMD:R_0603_1608Metric_Pad0.98x0.95mm_HandSolder
- R8: renamed from R30; footprint (none) -> Resistor_SMD:R_0603_1608Metric_Pad0.98x0.95mm_HandSolder
- R9: renamed from R15; footprint (none) -> Resistor_SMD:R_0603_1608Metric_Pad0.98x0.95mm_HandSolder
- SW2, SW3: footprint (none) -> Button_Switch_THT:SW_PUSH_6mm
- renumbered C6 to C3, D3 to D1, D5 to D4, D6 to D5, D7 to D6, D8 to D7, J2 to J1, J1 to J2, P2 to P1, R7 to R2, R8 to R4, U4 to U1, U8 to U2, U5 to U3, U6 to U4, U7 to U5
Connections:
- net +3.3V is gone; now on net +3V3: C8.1, C9.1, R13.2, R22.2, U3.3 (3V3)
- net BAT+ is gone; now on an unnamed net: SW1.1
- net Vout is gone; now on net +5V: C2.1, C5.1, D1.1 (K), R11.2, R2.1, U1.7 (BOOT)
- net +5V: now also D8.2 (A); no longer C13.1, C14.1, R24.1, U5.3 (VI)
- net at C4.1, U2.14 (V_{BAT}), U2.15 (V_{BAT})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: no longer J1.2 (Pin_2)
- net OUTVCC: no longer names the net of SW1.2
- net OUTVCC: now also J1.2 (Pin_2)
- new net: C13.1, C14.1, D8.1 (K), R24.1, U5.3 (VI)
- no-connect marks 9 -> 27
Other:
- note removed: "Ceramic Cap."
- note removed: "R3 set chargin current 10k = 130 ma"
- note removed: "TOODOO 5V afscheiden van VBUS, en achter Buckboost steken Vbussen naar 5V vervangen zodat het allemaal op batterij werkt"
- note removed: "USB C met een TP4056 om de herlaadbare batterij te regelen"
- company: (none) -> Jay D'Hulster
- title: (none) -> Biosensor
- moved on the sheet: C1, C10, C11, C12, C13, C14, C15, C16, C17, C18, C2, C3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

Commit message: update
Parts:
- removed SW1: SW_DIP_x01, Button_Switch_SMD:SW_DIP_SPSTx01_Slide_6.7x4.1mm_W8.61mm_P2.54mm_LowProfile, symbol Switch:SW_DIP_x01
- added SW1: SW_SPDT, Button_Switch_THT:SW_Slide_1P2T_CK_OS102011MS2Q, symbol Switch:SW_SPDT
- C1: footprint Capacitor_SMD:C_0603_1608Metric_Pad1.08x0.95mm_HandSolder -> 595D:CAP_595D-B_VSS
- C2: footprint Capacitor_SMD:C_0603_1608Metric_Pad1.08x0.95mm_HandSolder -> 595D:CAP_595D-C_VSS
- D1: value SS34 -> MBRS140T3; footprint Diode_SMD:D_SMA_Handsoldering -> Diode_SMD:D_SMB_Handsoldering
- L1: footprint Inductor_SMD:L_12x12mm_H8mm -> 595D:LPS4018223MRC
Connections:
- net at J1.2 (Pin_2): now also SW1.1 (A)
- net at C4.1, U2.14 (V_{BAT}), U2.15 (V_{BAT})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: now also SW1.2 (B)
- no-connect marks 27 -> 28
Changed lines of the file:
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@@
   (no_connect (at 107.95 196.85))
   (no_connect (at 259.08 73.66))
+  (no_connect (at 312.42 59.69))
   (no_connect (at 363.22 201.93))
   (no_connect (at 107.95 207.01))
@@
     (stroke (width 0) (type default))
   )
-  (wire (pts (xy 314.96 57.15) (xy 321.31 57.15))
+  (wire (pts (xy 312.42 54.61) (xy 321.31 54.61))
     (stroke (width 0) (type default))
   )
@@
     (stroke (width 0) (type default))
   )
-  (wire (pts (xy 293.37 57.15) (xy 299.72 57.15))
+  (wire (pts (xy 293.37 57.15) (xy 302.26 57.15))
     (stroke (width 0) (type default))
   )
@@
     (stroke (width 0) (type default))
   )
-  (wire (pts (xy 321.31 57.15) (xy 321.31 69.85))
+  (wire (pts (xy 321.31 54.61) (xy 321.31 69.85))
     (stroke (width 0) (type default))
   )
@@
       (effects (font (size 1.27 1.27)))
     )
-    (property "Value" "SS34" (at 423.2275 33.02 0)
-      (effects (font (size 1.27 1.27)))
-    )
-    (property "Footprint" "Diode_SMD:D_SMA_Handsoldering" (at 422.91 36.83 0)
+    (property "Value" "MBRS140T3" (at 423.2275 33.02 0)
+      (effects (font (size 1.27 1.27)))
+    )
+    (property "Footprint" "Diode_SMD:D_SMB_Handsoldering" (at 422.91 36.83 0)
       (effects (font (size 1.27 1.27)) hide)
     )
@@
       (effects (font (size 1.27 1.27)))
     )
-    (property "Footprint" "Inductor_SMD:L_12x12mm_H8mm" (at 406.4 48.26 0)
+    (property "Footprint" "595D:LPS4018223MRC" (at 406.4 48.26 0)
       (effects (font (size 1.27 1.27)) hide)
     )
@@
       (effects (font (size 1.27 1.27)) (justify left))
     )
-    (property "Footprint" "Capacitor_SMD:C_0603_1608Metric_Pad1.08x0.95mm_HandSolder" (at 468.63 52.07 0)
+    (property "Footprint" "595D:CAP_595D-C_VSS" (at 468.63 52.07 0)
       (effects (font (size 1.27 1.27)) hide)
     )
@@
     )
   )
+  (symbol (lib_id "Switch:SW_SPDT") (at 307.34 57.15 0) (unit 1)
+    (in_bom yes) (on_board yes) (dnp no) (fields_autoplaced)
+    (property "Reference" "SW1" (at 307.34 49.53 0)
+      (effects (font (size 1.27 1.27)))
+    )
+    (property "Value" "SW_SPDT" (at 307.34 52.07 0)
+      (effects (font (size 1.27 1.27)))
+    )
+    (property "Footprint" "Button_Switch_THT:SW_Slide_1P2T_CK_OS102011MS2Q" (at 307.34 57.15 0)
+      (effects (font (size 1.27 1.27)) hide)
+    )
+    (property "Datasheet" "~" (at 307.34 57.15 0)
+      (effects (font (size 1.27 1.27)) hide)
+    )
+    (pin "1")
+    (pin "2")
+    (pin "3")
+    (instances
+      (project "biosensor"
+        (path "/e63e39d7-6ac0-4ffd-8aa3-1841a4541b55"
+          (reference "SW1") (unit 1)
+        )
+      )
+    )
+  )
   (symbol (lib_id "power:GND") (at 274.32 166.37 0) (unit 1)
     (in_bom yes) (on_board yes) (dnp no) (fields_autoplaced)
@@
       (effects (font (size 1.27 1.27)) (justify left))
     )
-    (property "Footprint" "Capacitor_SMD:C_0603_1608Metric_Pad1.08x0.95mm_HandSolder" (at 392.43 52.07 0)
+    (property "Footprint" "595D:CAP_595D-B_VSS" (at 392.43 52.07 0)
       (effects (font (size 1.27 1.27)) hide)
     )
@@
         )
       )
-    )
-  )
-  (symbol (lib_id "Switch:SW_DIP_x01") (at 307.34 57.15 0) (unit 1)
-    (in_bom yes) (on_board yes) (dnp no) (fields_autoplaced)
-    (property "Reference" "SW1" (at 307.34 49.53 0)
-      (effects (font (size 1.27 1.27)))
-    )
-    (property "Value" "SW_DIP_x01" (at 307.34 52.07 0)
-      (effects (font (size 1.27 1.27)))
-    )
-    (property "Footprint" "Button_Switch_SMD:SW_DIP_SPSTx01_Slide_6.7x4.1mm_W8.61mm_P2.54mm_LowProfile" (at 307.34 57.15 0)
-      (effects (font (size 1.27 1.27)) hide)
-    )
-    (property "Datasheet" "~" (at 307.34 57.15 0)
-      (effects (font (size 1.27 1.27)) hide)
-    )
-    (pin "1")
-    (pin "2")
-    (instances
-      (project "biosensor"
-        (path "/e63e39d7-6ac0-4ffd-8aa3-1841a4541b55"
-          (reference "SW1") (unit 1)
-        )
-      )
